File: bare_varients/XY_Faces/solar-panel-NoCutout.kicad_pcb (KiCad board)
At the start: 4 copper layers, 83 x 98 mm, 25 parts, among them J1 CON-5040500591, J2 Conn_01x01, J3 Conn_01x01, J4 Conn_01x01, J5 Conn_01x01, U1 VEML7700, U2 MCP9808_DFN, U3 DRV2605LDGS

Commit message: Added the old Pleiades Five Logo
Parts:
- added G***: LOGO, LOGO, F.Cu at (158.0, 92.3)
- added G***: LOGO, LOGO, F.Cu at (169.8, 129.3)
- added G***: LOGO, LOGO, F.Cu at (145.3, 92.7)
- added G***: LOGO, LOGO, F.Cu at (145.6, 101.4)
- added G***: LOGO, LOGO, F.Cu at (152.2, 96.7)
- added G***: LOGO, LOGO, F.Cu at (135.0, 96.1)
- added G***: LOGO, LOGO, F.Cu at (157.7, 101.6)
Other:
- board text added: "Ad Astra Tempore"
- board text added: "BRONCO SPACE Educational Product For Instructional Use Only"
- board text added: "THE PLEIADES FIVE"
- board text added: "The PROVES Kit V1.5"
