File: Z_Face_V2/Z_Face_V2.kicad_pcb (KiCad board)
At the start: 4 copper layers, 100 x 100 mm, 45 parts, among them J1 CON-5040500591, J2 Screw_Terminal_01x02, J3 Screw_Terminal_01x02, J4 Conn_01x01, J5 Conn_01x01, J6 Conn_01x01, J7 Conn_01x01, U1 VEML7700, U2 DRV2605LDGS, U3 MCP9808_DFN, U4 AD8495, U5 ADS1015IDGS, U6 TLVH431 DBZ SOT-23

Commit message: Z- Removed Thermocouple
Parts:
- removed C10, C7: 0.1uF, Capacitor_SMD:C_0805_2012Metric
- removed C4: 1uF, Capacitor_SMD:C_0805_2012Metric
- removed C5, C6: 0.01uF, Capacitor_SMD:C_0805_2012Metric
- removed C8, C9: 10uF, Capacitor_SMD:C_0805_2012Metric
- removed FB1, FB2, FB3: FerriteBead, Resistor_SMD:R_0603_1608Metric
- removed J2: Screw_Terminal_01x02, SolarPanelBoards:ScrewTerminal
- removed J3: Screw_Terminal_01x02, TerminalBlock:TerminalBlock_bornier-2_P5.08mm
- removed JP1: SolderJumper_2_Open, Jumper:SolderJumper-2_P1.3mm_Open_RoundedPad1.0x1.5mm
- removed R2: 1-MOhm, Resistor_SMD:R_0603_1608Metric
- removed R3, R4: 100-Ohm, Resistor_SMD:R_0603_1608Metric
- removed R5: 1k, Resistor_SMD:R_0603_1608Metric
- removed R6: 10k-Ohm, Resistor_SMD:R_0603_1608Metric
- removed U4: AD8495, Package_SO:MSOP-8_3x3mm_P0.65mm
- removed U5: ADS1015IDGS, Package_SO:TSSOP-10_3x3mm_P0.5mm
- removed U6: TLVH431 DBZ SOT-23, Package_TO_SOT_SMD:SOT-23
Routing:
- net SCL: track 64.7 -> 44.8 mm, vias 2 -> 1
- net SDA: track 70.4 -> 52.3 mm
- net AVDD: track 17.2 -> 0.00 mm
- net Net-(C4-Pad1): track 16.9 -> 0.00 mm
- net GND: track 61.3 -> 45.0 mm, vias 11 -> 10
- net OUT: track 16.1 -> 0.00 mm
- net AGND: track 15.7 -> 0.00 mm, vias 2 -> 0
- net Net-(J2-Pad2): track 15.2 -> 0.00 mm
- net Net-(C5-Pad2): track 12.0 -> 0.00 mm
- net Net-(C6-Pad1): track 11.9 -> 0.00 mm
- net Net-(J2-Pad1): track 11.7 -> 0.00 mm
- net +3V3: track 41.6 -> 32.6 mm, vias 5 -> 2
- net Net-(R5-Pad1): track 8.63 -> 0.00 mm
- net Net-(JP1-Pad1): track 4.00 -> 0.00 mm
Other:
- board text removed: "For Instructional Use Only."
- board text removed: "SOLIDWORKS Educational Product."
