File: Z_Face_V2/Z_Face_V2.kicad_sch (KiCad schematic)
At the start: 45 parts, among them J1 CON-5040500591, J2 Screw_Terminal_01x02, J3 Screw_Terminal_01x02, J4 Conn_01x01, J5 Conn_01x01, J6 Conn_01x01, J7 Conn_01x01, U1 VEML7700, U2 DRV2605LDGS, U3 MCP9808_DFN, U4 AD8495, U5 ADS1015IDGS, U6 TLVH431 DBZ SOT-23

Commit message: Z- Removed Thermocouple
Parts:
- removed C10, C7: 0.1uF, Capacitor_SMD:C_0805_2012Metric, symbol Device:C
- removed C4: 1uF, Capacitor_SMD:C_0805_2012Metric, symbol Device:C
- removed C5, C6: 0.01uF, Capacitor_SMD:C_0805_2012Metric, symbol Device:C
- removed C8, C9: 10uF, Capacitor_SMD:C_0805_2012Metric, symbol Device:C
- removed FB1, FB2, FB3: FerriteBead, Resistor_SMD:R_0603_1608Metric, symbol Device:FerriteBead
- removed J2: Screw_Terminal_01x02, SolarPanelBoards:ScrewTerminal, symbol Connector:Screw_Terminal_01x02
- removed J3: Screw_Terminal_01x02, TerminalBlock:TerminalBlock_bornier-2_P5.08mm, symbol Connector:Screw_Terminal_01x02
- removed JP1: SolderJumper_2_Open, Jumper:SolderJumper-2_P1.3mm_Open_RoundedPad1.0x1.5mm, symbol Jumper:SolderJumper_2_Open
- removed R2: 1-MOhm, Resistor_SMD:R_0603_1608Metric, symbol Device:R_US
- removed R3, R4: 100-Ohm, Resistor_SMD:R_0603_1608Metric, symbol Device:R_US
- removed R5: 1k, Resistor_SMD:R_0603_1608Metric, symbol Device:R_US
- removed R6: 10k-Ohm, Resistor_SMD:R_0603_1608Metric, symbol Device:R_US
- removed U4: AD8495, Package_SO:MSOP-8_3x3mm_P0.65mm, symbol Sensor_Temperature:AD8495
- removed U5: ADS1015IDGS, Package_SO:TSSOP-10_3x3mm_P0.5mm, symbol Analog_ADC:ADS1015IDGS
- removed U6: TLVH431 DBZ SOT-23, Package_TO_SOT_SMD:SOT-23, symbol Reference_Voltage:TL431DBZ
Connections:
- no-connect marks 9 -> 8
Other:
- note removed: "Default I2C: 0x48"
- note removed: "Jumped I2C: 0x49"
- moved on the sheet: D1, D2, D3, D4, J1, J4, J5, J6, J7, R1, SC1, SC2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
