File: Z_Face_V3/Z_Face_V3.kicad_sch (KiCad schematic)
At the start: 33 parts, among them J1 Molex FC Connection, J2 DF11 FC Connection, J4 Conn_01x01, J5 Conn_01x01, J6 Conn_01x01, J7 Conn_01x01, U1 VEML7700, U2 DRV2605LDGS, U4 TCA4311A, U5 TMP112xxDRL

Commit message: Z- V3: Nearly Completed Layout
Connections:
- net +3V3: now also C5.1, R2.1, R3.1, R4.1, R5.1, U4.8 (VCC)
Changed lines of the file:
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@@
 	(wire
 		(pts
+			(xy 93.98 38.1) (xy 93.98 49.53)
+		)
+		(stroke
+			(width 0)
+			(type default)
+		)
+	)
+	(wire
+		(pts
 			(xy 82.55 82.55) (xy 93.98 82.55)
 		)
@@
 					(unit 1)
 				)
+			)
+		)
+	)
+	(symbol
+		(lib_id "solar-panel-side-Z-rescue:+3.3V-power")
+		(at 93.98 38.1 0)
+		(unit 1)
+		(exclude_from_sim no)
+		(in_bom yes)
+		(on_board yes)
+		(dnp no)
+		(property "Reference" "#PWR024"
+			(at 93.98 41.91 0)
+			(effects
+				(font
+					(size 1.27 1.27)
+				)
+				(hide yes)
+			)
+		)
+		(property "Value" "+3V3"
+			(at 94.361 33.7058 0)
+			(effects
+				(font
+					(size 1.27 1.27)
+				)
+			)
+		)
+		(property "Footprint" ""
+			(at 93.98 38.1 0)
+			(effects
+				(font
+					(size 1.27 1.27)
+				)
+				(hide yes)
+			)
+		)
+		(property "Datasheet" ""
+			(at 93.98 38.1 0)
+			(effects
+				(font
+					(size 1.27 1.27)
+				)
+				(hide yes)
+			)
+		)
+		(property "Description" ""
+			(at 93.98 38.1 0)
+			(effects
+				(font
+					(size 1.27 1.27)
+				)
+			)
+		)
+		(pin "1"
+		)
+		(instances
+			(project "Z_Face_V3"
+				(path "/b92e10d4-ef16-4e79-8a94-1185be6812fd"
+					(reference "#PWR024")
+					(unit 1)
+				)

Commit message: V3: As Ordered Sept 25, 2025
Parts:
- removed U1: VEML7700, VEML7700-TT:XDCR_VEML7700-TT, symbol Adafruit VEML7700-eagle-import:VEML7700
- added U1: VEML6031X00, easyeda2kicad:SENSOR-SMD_VEML6031X00, symbol easyeda2kicad:VEML6031X00
Connections:
- net +3V3: now also U1.6 (VDD)
- net GND: now also U1.1 (GND), U1.4 (GND)
- net SCL: now also U1.5 (SCL)
- net SDA: now also U1.2 (SDA)
- no-connect marks 5 -> 6
Other:
- company: CPP BroncoSpace -> Open Source Space Foundation
Changed lines of the file:
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@@
 	(title_block
 		(title "Solar Panel Board -Z")
-		(date "2023-03-20")
+		(date "2025-09-25")
 		(rev "V3")
-		(company "CPP BroncoSpace")
+		(company "Open Source Space Foundation")
 	)
 	(text "Light Sensor"
@@
 	)
 	(junction
-		(at 205.74 17.78)
+		(at 205.74 25.4)
 		(diameter 0)
 		(color 0 0 0 0)
@@
 	)
 	(junction
-		(at 205.74 50.8)
+		(at 205.74 43.18)
 		(diameter 0)
 		(color 0 0 0 0)
@@
 	)
 	(no_connect
+		(at 214.63 34.29)
+	)
+	(no_connect
 		(at 33.02 146.05)
 	)
@@
 	(wire
 		(pts
-			(xy 205.74 17.78) (xy 228.6 17.78)
+			(xy 205.74 25.4) (xy 228.6 25.4)
 		)
 		(stroke
@@
 	(wire
 		(pts
-			(xy 205.74 16.51) (xy 205.74 17.78)
+			(xy 205.74 24.13) (xy 205.74 25.4)
 		)
 		(stroke
@@
 	(wire
 		(pts
-			(xy 157.48 69.85) (xy 157.48 36.83)
+			(xy 157.48 69.85) (xy 157.48 35.56)
 		)
 		(stroke
@@
 	(wire
 		(pts
-			(xy 228.6 38.1) (xy 228.6 50.8)
+			(xy 228.6 38.1) (xy 228.6 43.18)
 		)
 		(stroke
@@
 	(wire
 		(pts
-			(xy 157.48 36.83) (xy 190.5 36.83)
+			(xy 157.48 35.56) (xy 196.85 35.56)
 		)
 		(stroke
@@
 	(wire
 		(pts
-			(xy 152.4 31.75) (xy 190.5 31.75)
+			(xy 152.4 33.02) (xy 196.85 33.02)
 		)
 		(stroke
@@
 	(wire
 		(pts
-			(xy 205.74 17.78) (xy 205.74 19.05)
+			(xy 205.74 25.4) (xy 205.74 26.67)
 		)
 		(stroke
@@
 	(wire
 		(pts
-			(xy 228.6 50.8) (xy 205.74 50.8)
+			(xy 228.6 43.18) (xy 205.74 43.18)
 		)
 		(stroke
@@
 	(wire
 		(pts
-			(xy 152.4 67.31) (xy 152.4 31.75)
+			(xy 152.4 67.31) (xy 152.4 33.02)
 		)
 		(stroke
@@
 	(wire
 		(pts
-			(xy 205.74 49.53) (xy 205.74 50.8)
+			(xy 205.74 41.91) (xy 205.74 43.18)
 		)
 		(stroke
@@
 	(wire
 		(pts
-			(xy 205.74 50.8) (xy 205.74 52.07)
+			(xy 205.74 43.18) (xy 205.74 44.45)
 		)
 		(stroke
@@
 	(wire
 		(pts
-			(xy 228.6 17.78) (xy 228.6 30.48)
+			(xy 228.6 25.4) (xy 228.6 30.48)
 		)
 		(stroke
@@
 	)
 	(symbol
-		(lib_id "Adafruit VEML7700-eagle-import:VEML7700")
-		(at 205.74 34.29 0)
-		(unit 1)
-		(exclude_from_sim no)
-		(in_bom yes)
-		(on_board yes)
-		(dnp no)
-		(property "Reference" "U1"
-			(at 208.28 24.13 0)
-			(effects
-				(font
-					(size 2.54 2.159)
-				)
-				(justify left bottom)
-			)
-		)
-		(property "Value" "VEML7700"
-			(at 205.74 34.29 0)
-			(effects
-				(font
-					(size 1.27 1.27)
-				)
-				(hide yes)
-			)
-		)
-		(property "Footprint" "VEML7700-TT:XDCR_VEML7700-TT"
-			(at 205.74 34.29 0)
-			(effects
-				(font
-					(size 1.27 1.27)
-				)
-				(hide yes)
-			)
-		)
-		(property "Datasheet" ""
-			(at 205.74 34.29 0)
-			(effects
-				(font
-					(size 1.27 1.27)
-				)
-				(hide yes)
-			)
-		)
-		(property "Description" ""
-			(at 205.74 34.29 0)
-			(effects
-				(font
-					(size 1.27 1.27)
-				)
-			)
-		)
-		(pin "1"
-		)
-		(pin "2"
-		)
-		(pin "3"
-		)
-		(pin "4"
-		)
-		(instances
-			(project ""
-				(path "/b92e10d4-ef16-4e79-8a94-1185be6812fd"
-					(reference "U1")
-					(unit 1)
-				)
-			)
-		)
-	)
-	(symbol
 		(lib_id "solar-panel-side-Z-rescue:+3.3V-power")
 		(at 49.53 69.85 0)
@@
 		(lib_name "GND_1")
 		(lib_id "power:GND")
-		(at 205.74 52.07 0)
+		(at 205.74 44.45 0)
 		(unit 1)
 		(exclude_from_sim no)
@@
 		(fields_autoplaced yes)
 		(property "Reference" "#PWR08"
-			(at 205.74 58.42 0)
+			(at 205.74 50.8 0)
 			(effects
 				(font
@@
 		)
 		(property "Value" "GND"
-			(at 205.74 57.15 0)
+			(at 205.74 49.53 0)
 			(effects
 				(font
@@
 		)
 		(property "Footprint" ""
-			(at 205.74 52.07 0)
+			(at 205.74 44.45 0)
 			(effects
 				(font
@@
 		)
 		(property "Datasheet" ""
-			(at 205.74 52.07 0)
+			(at 205.74 44.45 0)
 			(effects
 				(font
@@
 		)
 		(property "Description" "Power symbol creates a global label with name \"GND\" , ground"
-			(at 205.74 52.07 0)
+			(at 205.74 44.45 0)
 			(effects
 				(font
@@
 	)
 	(symbol
+		(lib_id "easyeda2kicad:VEML6031X00")
+		(at 205.74 34.29 0)
+		(unit 1)
+		(exclude_from_sim no)
+		(in_bom yes)
+		(on_board yes)
+		(dnp no)
+		(fields_autoplaced yes)
+		(property "Reference" "U1"
+			(at 219.71 27.8698 0)
+			(effects
+				(font
+					(size 1.27 1.27)
+				)
+			)
+		)
+		(property "Value" "VEML6031X00"
+			(at 219.71 30.4098 0)
+			(effects
+				(font
+					(size 1.27 1.27)
+				)
+			)
+		)
+		(property "Footprint" "easyeda2kicad:SENSOR-SMD_VEML6031X00"
+			(at 205.74 44.45 0)
+			(effects
+				(font
+					(size 1.27 1.27)
+				)
+				(hide yes)
+			)
+		)
+		(property "Datasheet" ""
+			(at 205.74 34.29 0)
+			(effects
+				(font
+					(size 1.27 1.27)
+				)
+				(hide yes)
+			)
+		)
+		(property "Description" ""
+			(at 205.74 34.29 0)
+			(effects
+				(font
+					(size 1.27 1.27)
+				)
+				(hide yes)
+			)
+		)
+		(property "LCSC Part" "C3678616"
+			(at 205.74 46.99 0)
+			(effects
+				(font
+					(size 1.27 1.27)
+				)
+				(hide yes)
+			)
+		)
+		(pin "5"
+		)
+		(pin "1"
+		)
+		(pin "4"
+		)
+		(pin "6"
+		)
+		(pin "3"
+		)
+		(pin "2"
+		)
+		(instances
+			(project ""
+				(path "/b92e10d4-ef16-4e79-8a94-1185be6812fd"
+					(reference "U1")
+					(unit 1)
+				)
+			)
+		)
+	)
+	(symbol
 		(lib_name "GND_1")
 		(lib_id "power:GND")
@@
 	(symbol
 		(lib_id "solar-panel-side-Z-rescue:+3.3V-power")
-		(at 205.74 16.51 0)
+		(at 205.74 24.13 0)
 		(unit 1)
 		(exclude_from_sim no)
@@
 		(dnp no)
 		(property "Reference" "#PWR0102"
-			(at 205.74 20.32 0)
+			(at 205.74 27.94 0)
 			(effects
 				(font
@@
 		)
 		(property "Value" "+3V3"
-			(at 201.422 14.478 0)
+			(at 201.422 22.098 0)
 			(effects
 				(font
@@
 		)
 		(property "Footprint" ""
-			(at 205.74 16.51 0)
+			(at 205.74 24.13 0)
 			(effects
 				(font
@@
 		)
 		(property "Datasheet" ""
-			(at 205.74 16.51 0)
+			(at 205.74 24.13 0)
 			(effects
 				(font
@@
 		)
 		(property "Description" ""
-			(at 205.74 16.51 0)
+			(at 205.74 24.13 0)
 			(effects
 				(font
